File: boards/terminal/terminal.kicad_pcb (KiCad board)
At the start: 2 copper layers, 108 parts, among them J1 Conn_01x14, J2 Conn_01x14, SW1 SW_Push_45deg, SW10 SW_Push_45deg, SW11 SW_Push_45deg, SW12 SW_Push_45deg, SW13 SW_Push_45deg, SW14 SW_Push_45deg, SW15 SW_Push_45deg, SW16 SW_Push_45deg, SW17 SW_Push_45deg, SW18 SW_Push_45deg, SW19 SW_Push_45deg, SW2 SW_Push_45deg, SW20 SW_Push_45deg, SW21 SW_Push_45deg, SW22 SW_Push_45deg, SW23 SW_Push_45deg, SW24 SW_Push_45deg, SW25 SW_Push_45deg, SW26 SW_Push_45deg, SW27 SW_Push_45deg, SW28 SW_Push_45deg, SW29 SW_Push_45deg, SW3 SW_Push_45deg, SW30 SW_Push_45deg, SW31 SW_Push_45deg, SW32 SW_Push_45deg, SW33 SW_Push_45deg, SW34 SW_Push_45deg, SW35 SW_Push_45deg, SW36 SW_Push_45deg, SW37 SW_Push_45deg, SW38 SW_Push_45deg, SW39 SW_Push_45deg, SW4 SW_Push_45deg, SW40 SW_Push_45deg, SW41 SW_Push_45deg, SW42 SW_Push_45deg, SW43 SW_Push_45deg, SW44 SW_Push_45deg, SW45 SW_Push_45deg, SW46 SW_Push_45deg, SW47 SW_Push_45deg, SW48 SW_Push_45deg, SW49 SW_Push_45deg, SW5 SW_Push_45deg, SW50 SW_Push_45deg, SW51 SW_Push_45deg, SW52 SW_Push_45deg, SW53 SW_Push_45deg, SW54 SW_Push_45deg, SW55 SW_Push_45deg, SW56 SW_Push_45deg, SW57 SW_Push_45deg, SW58 SW_Push_45deg, SW59 SW_Push_45deg, SW6 SW_Push_45deg, SW60 SW_Push_45deg, SW61 SW_Push_45deg, SW62 SW_Push_45deg, SW63 SW_Push_45deg, SW64 SW_Push_45deg, SW65 SW_Push_45deg, SW66 SW_Push_45deg, SW67 SW_Push_45deg, SW68 SW_Push_45deg, SW69 SW_Push_45deg, SW7 SW_Push_45deg, SW70 SW_Push_45deg, SW71 SW_Push_45deg, SW72 SW_Push_45deg, SW73 SW_Push_45deg, SW74 SW_Push_45deg, SW76 SW_Push_45deg, SW77 SW_Push_45deg, SW78 SW_Push_45deg, SW79 SW_Push_45deg, SW8 SW_Push_45deg, SW80 SW_Push_45deg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

Commit message: Fix keyboard layout
Parts:
- added SW75: FN, Button_Switch_Keyboard:SW_Cherry_MX_1.00u_PCB, F.Cu at (291.0, 118.0)
- SW1: value SW_Push_45deg -> ESC
- SW10: value SW_Push_45deg -> A
- SW11, SW71: value SW_Push_45deg -> \
- SW12: value SW_Push_45deg -> WIN
- SW13: value SW_Push_45deg -> F2
- SW14: value SW_Push_45deg -> 2
- SW15: value SW_Push_45deg -> W
- SW16: value SW_Push_45deg -> S
- SW17: value SW_Push_45deg -> Z
- SW18: value SW_Push_45deg -> ALT
- SW19: value SW_Push_45deg -> F3
- SW2: value SW_Push_45deg -> ~`
- SW20: value SW_Push_45deg -> 3
- SW21: value SW_Push_45deg -> E
- SW22: value SW_Push_45deg -> D
- SW23: value SW_Push_45deg -> X
- SW24: value SW_Push_45deg -> SPACE
- SW25: value SW_Push_45deg -> F4
- SW26: value SW_Push_45deg -> 4
- SW27: value SW_Push_45deg -> R
- SW28: value SW_Push_45deg -> F
- SW29: value SW_Push_45deg -> C
- SW3: value SW_Push_45deg -> TAB
- SW30: value SW_Push_45deg -> ALT; footprint Button_Switch_Keyboard:SW_Cherry_MX_1.50u_PCB -> Button_Switch_Keyboard:SW_Cherry_MX_1.25u_PCB
- SW31: value SW_Push_45deg -> F5
- SW32: value SW_Push_45deg -> 5
- SW33: value SW_Push_45deg -> T
- SW34: value SW_Push_45deg -> G
- SW35: value SW_Push_45deg -> V
- SW36: value SW_Push_45deg -> MENU; footprint Button_Switch_Keyboard:SW_Cherry_MX_1.50u_PCB -> Button_Switch_Keyboard:SW_Cherry_MX_1.25u_PCB
- SW37: value SW_Push_45deg -> F6
- SW38: value SW_Push_45deg -> 6
- SW39: value SW_Push_45deg -> Y
- SW4: value SW_Push_45deg -> CAPS
- SW40: value SW_Push_45deg -> H
- SW41: value SW_Push_45deg -> B
- SW42: value SW_Push_45deg -> CTRL; footprint Button_Switch_Keyboard:SW_Cherry_MX_1.50u_PCB -> Button_Switch_Keyboard:SW_Cherry_MX_1.25u_PCB
- SW43: value SW_Push_45deg -> F7
- SW44: value SW_Push_45deg -> 7
- SW45: value SW_Push_45deg -> U
- SW46: value SW_Push_45deg -> J
- SW47: value SW_Push_45deg -> N
- SW48: value SW_Push_45deg -> F8
- SW49: value SW_Push_45deg -> 8
- SW5, SW72: value SW_Push_45deg -> SHIFT
- SW50: value SW_Push_45deg -> I
- SW51: value SW_Push_45deg -> K
- SW52: value SW_Push_45deg -> M
- SW53: value SW_Push_45deg -> F9
- SW54: value SW_Push_45deg -> 9
- SW55: value SW_Push_45deg -> O
- SW56: value SW_Push_45deg -> L
- SW57: value SW_Push_45deg -> ,
- SW58: value SW_Push_45deg -> F10
- SW59: value SW_Push_45deg -> 0
- SW6: value SW_Push_45deg -> CTRL
- SW60: value SW_Push_45deg -> P
- SW61: value SW_Push_45deg -> ;
- SW62: value SW_Push_45deg -> .
- SW63: value SW_Push_45deg -> F11
- SW64: value SW_Push_45deg -> -
- SW65: value SW_Push_45deg -> [
- SW66: value SW_Push_45deg -> '
- SW67: value SW_Push_45deg -> /
- SW68: value SW_Push_45deg -> F12
- SW69: value SW_Push_45deg -> =
- SW7: value SW_Push_45deg -> F1
- SW70: value SW_Push_45deg -> ]
- SW73: value SW_Push_45deg -> BACKSPACE
- SW74: value SW_Push_45deg -> ENTER
- SW76: value SW_Push_45deg -> PRINT_SCR
- SW77: value SW_Push_45deg -> INS
- SW78: value SW_Push_45deg -> DEL
- SW79: value SW_Push_45deg -> LEFT
- SW8: value SW_Push_45deg -> 1
- SW80: value SW_Push_45deg -> SCROLL_LOCK
- SW81: value SW_Push_45deg -> HOME
- SW82: value SW_Push_45deg -> END
- SW83: value SW_Push_45deg -> UP
- SW84: value SW_Push_45deg -> DOWN
- SW85: value SW_Push_45deg -> PAUSE
- SW86: value SW_Push_45deg -> PG_UP
- SW87: value SW_Push_45deg -> PG_DOWN
- SW88: value SW_Push_45deg -> RIGHT
- SW9: value SW_Push_45deg -> Q
- moved J1 373.4 mm to (35.4, 204.1)
- moved J2 373.4 mm to (24.2, 215.1)
- moved U1 373.4 mm to (189.6, 189.0)
- moved U2 373.4 mm to (25.3, 164.5)
- moved D17 226.7 mm to (414.1, -4.40)
- moved SW86 67.4 mm to (354.0, 42.0)
- moved SW81 64.0 mm to (335.0, 42.0)
- moved SW88 63.4 mm to (354.0, 118.0)
- moved SW85 62.8 mm to (354.0, 17.0)
- moved SW77 62.6 mm to (316.0, 42.0)
- moved SW83 61.4 mm to (335.0, 99.0)
- moved SW87 60.6 mm to (354.0, 61.0)
- moved SW84 60.5 mm to (335.0, 118.0)
- moved SW80 59.4 mm to (335.0, 17.0)
- moved SW82 57.7 mm to (335.0, 61.0)
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Connections:
- SW4 pad 2: Net-(SW4-Pad2) -> Net-(SW10-Pad2)
- SW5 pad 2: Net-(SW5-Pad2) -> Net-(SW11-Pad2)
- SW6 pad 2: Net-(SW6-Pad2) -> Net-(SW12-Pad2)
