File: boards/keyboard/keyboard.kicad_pcb (KiCad board)
At the start: 2 copper layers, 177 parts, among them J1 Conn_02x13_Odd_Even, SW1 ESC, SW10 A, SW11 \, SW12 WIN, SW13 F2, SW14 2, SW15 W, SW16 S, SW17 Z, SW18 ALT, SW19 F3, SW2 ~`, SW20 3, SW21 E, SW22 D, SW23 X, SW24 SPACE, SW25 F4, SW26 4, SW27 R, SW28 F, SW29 C, SW3 TAB, SW30 ALT, SW31 F5, SW32 5, SW33 T, SW34 G, SW35 V, SW36 MENU, SW37 F6, SW38 6, SW39 Y, SW4 CAPS, SW40 H, SW41 B, SW42 CTRL, SW43 F7, SW44 7, SW45 U, SW46 J, SW47 N, SW48 F8, SW49 8, SW5 SHIFT, SW50 I, SW51 K, SW52 M, SW53 F9, SW54 9, SW55 O, SW56 L, SW57 ,, SW58 F10, SW59 0, SW6 CTRL, SW60 P, SW61 ;, SW62 ., SW63 F11, SW64 -, SW65 [, SW66 ', SW67 /, SW68 F12, SW69 =, SW7 F1, SW70 ], SW71 \, SW72 SHIFT, SW73 BACKSPACE, SW74 ENTER, SW75 FN, SW76 PRINT_SCR, SW77 INS, SW78 DEL, SW79 LEFT, SW8 1, SW80 SCROLL_LOCK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

Commit message: Add production files, fix licensing
Parts:
- added D89: LED, LED_SMD:LED_1206_3216Metric_Castellated, F.Cu at (331.7, 57.0)
- added D90: LED, LED_SMD:LED_1206_3216Metric_Castellated, F.Cu at (350.7, 57.0)
- added D91: LED, LED_SMD:LED_1206_3216Metric_Castellated, F.Cu at (369.7, 57.0)
- added G***: LOGO, keyboard:softwareless_logo58x8, F.Cu at (350.7, 107.8)
- added R1: 330R, Resistor_SMD:R_0603_1608Metric_Pad1.05x0.95mm_HandSolder, F.Cu at (337.0, 56.1)
- added R2: 330R, Resistor_SMD:R_0603_1608Metric_Pad1.05x0.95mm_HandSolder, F.Cu at (356.0, 56.1)
- added R3: 330R, Resistor_SMD:R_0603_1608Metric_Pad1.05x0.95mm_HandSolder, F.Cu at (375.1, 56.2)
- added REF**: KiCad-Logo2_5mm_SilkScreen, Symbol:KiCad-Logo2_5mm_SilkScreen, B.Cu at (370.4, 110.5)
- added REF**: MountingHole_3.2mm_M3, MountingHole:MountingHole_3.2mm_M3, F.Cu at (125.2, 149.6)
- added REF**: MountingHole_3.2mm_M3, MountingHole:MountingHole_3.2mm_M3, F.Cu at (36.2, 107.6)
- added REF**: MountingHole_3.2mm_M3, MountingHole:MountingHole_3.2mm_M3, F.Cu at (372.7, 129.6)
- added REF**: MountingHole_3.2mm_M3, MountingHole:MountingHole_3.2mm_M3, F.Cu at (331.7, 129.6)
- added REF**: MountingHole_3.2mm_M3, MountingHole:MountingHole_3.2mm_M3, F.Cu at (300.0, 56.5)
- added REF**: MountingHole_3.2mm_M3, MountingHole:MountingHole_3.2mm_M3, F.Cu at (34.2, 57.1)
- added REF**: OSHW-Symbol_6.7x6mm_SilkScreen, Symbol:OSHW-Symbol_6.7x6mm_SilkScreen, B.Cu at (330.4, 111.8)
- added REF**: MountingHole_3.2mm_M3, MountingHole:MountingHole_3.2mm_M3, F.Cu at (319.0, 152.5)
- added REF**: MountingHole_3.2mm_M3, MountingHole:MountingHole_3.2mm_M3, F.Cu at (34.5, 152.0)
- added REF**: MountingHole_3.2mm_M3, MountingHole:MountingHole_3.2mm_M3, F.Cu at (115.5, 98.0)
- added REF**: MountingHole_3.2mm_M3, MountingHole:MountingHole_3.2mm_M3, F.Cu at (211.5, 97.5)
- added REF**: MountingHole_3.2mm_M3, MountingHole:MountingHole_3.2mm_M3, F.Cu at (269.5, 129.6)
- added REF**: MountingHole_3.2mm_M3, MountingHole:MountingHole_3.2mm_M3, F.Cu at (310.2, 129.6)
- added REF**: MountingHole_3.2mm_M3, MountingHole:MountingHole_3.2mm_M3, F.Cu at (205.2, 150.6)
- moved D67 29.4 mm to (277.0, 41.0), turned to 270 degrees
- moved D70 29.1 mm to (292.4, 102.7)
- moved D71 29.1 mm to (306.3, 121.7)
- moved D83 29.1 mm to (360.2, 121.7)
- moved D39 29.1 mm to (176.6, 140.7)
- moved D18 29.1 mm to (107.1, 140.7)
- moved D12 29.1 mm to (83.4, 140.7)
- moved D26 29.1 mm to (135.7, 83.7)
- moved D27 29.1 mm to (140.4, 102.7)
- moved D32 29.1 mm to (159.4, 102.7)
- moved D34 29.1 mm to (164.1, 39.7)
- moved D35 29.1 mm to (164.1, 64.7)
- moved D46 29.1 mm to (202.2, 64.7)
- moved D48 29.1 mm to (216.4, 102.7)
- moved D50 29.1 mm to (221.2, 39.7)
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Connections:
- J1 pad 23: Net-(J1-Pad23) -> /LED1
- J1 pad 24: Net-(J1-Pad24) -> /LED2
- J1 pad 25: Net-(J1-Pad25) -> /LED3
- J1 pad 26: Net-(J1-Pad26) -> GND
Routing:
- net GND: track 0.00 -> 68.5 mm, vias 0 -> 5
- net /LED3: track 0.00 -> 58.0 mm, vias 0 -> 1
- net /LED2: track 0.00 -> 45.1 mm, vias 0 -> 1
- net /LED1: track 0.00 -> 24.2 mm, vias 0 -> 1
- net /C14: track 117.7 -> 102.7 mm
- net /C15: track 163.1 -> 150.0 mm
- net /C8: track 498.4 -> 503.7 mm
- net /C6: track 583.1 -> 587.9 mm
- net /C9: track 451.5 -> 455.7 mm
- net Net-(D91-Pad1): track 0.00 -> 4.02 mm
- net /C12: track 157.5 -> 161.4 mm
- net Net-(D90-Pad1): track 0.00 -> 3.92 mm
- net Net-(D89-Pad1): track 0.00 -> 3.90 mm
- net /C16: track 167.4 -> 163.6 mm
- net /C10: track 357.5 -> 360.6 mm
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Other:
- board outline added: 350 x 122 mm
- board text added: "2022-03-22"
- board text added: "Licensed under CERN-OHL-P v2 or later"
- board text added: "github.com/Aifryz/softwareless"
