File: boards/keyboard/keyboard.sch (KiCad schematic (older format))
At the start: 177 parts, among them J1 Conn_02x13_Odd_Even, SW1 ESC, SW10 A, SW11 \\, SW12 WIN, SW13 F2, SW14 2, SW15 W, SW16 S, SW17 Z, SW18 ALT, SW19 F3, SW2 ~`, SW20 3, SW21 E, SW22 D, SW23 X, SW24 SPACE, SW25 F4, SW26 4, SW27 R, SW28 F, SW29 C, SW3 TAB, SW30 ALT, SW31 F5, SW32 5, SW33 T, SW34 G, SW35 V, SW36 MENU, SW37 F6, SW38 6, SW39 Y, SW4 CAPS, SW40 H, SW41 B, SW42 CTRL, SW43 F7, SW44 7, SW45 U, SW46 J, SW47 N, SW48 F8, SW49 8, SW5 SHIFT, SW50 I, SW51 K, SW52 M, SW53 F9, SW54 9, SW55 O, SW56 L, SW57 ,, SW58 F10, SW59 0, SW6 CTRL, SW60 P, SW61 ;, SW62 ., SW63 F11, SW64 -, SW65 [, SW66 ', SW67 /, SW68 F12, SW69 =, SW7 F1, SW70 ], SW71 \\, SW72 SHIFT, SW73 BACKSPACE, SW74 ENTER, SW75 FN, SW76 PRINT_SCR, SW77 INS, SW78 DEL, SW79 LEFT, SW8 1, SW80 SCROLL_LOCK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

Commit message: Add production files, fix licensing
Parts:
- added D89, D90, D91: LED, LED_SMD:LED_1206_3216Metric_Castellated, symbol Device:LED
- added R1, R2, R3: 330R, Resistor_SMD:R_0603_1608Metric_Pad1.05x0.95mm_HandSolder, symbol Device:R_Small
Connections:
- net LED1: now reaches J1.23 (Pin_23)
- net LED1: now also D89.2 (A)
- net LED2: now reaches J1.24 (Pin_24)
- net LED2: now also D90.2 (A)
- net LED3: now reaches J1.25 (Pin_25)
- net LED3: now also D91.2 (A)
- net GND: now reaches J1.26 (Pin_26)
- net GND: now also R1.1, R2.1, R3.1
- new net: D89.1 (K), R1.2
- new net: D90.1 (K), R2.2
- new net: D91.1 (K), R3.2
Other:
- moved on the sheet: D1, D10, D11, D12, D13, D14, D15, D16, D17, D18, D19, D2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
