File: boards/led_display/led_display.kicad_pcb (KiCad board)
At the start: 2 copper layers, 16 parts

Commit message: Add partial led board layout
Parts:
- added C1: 1u, Capacitor_SMD:C_0805_2012Metric, F.Cu at (200.2, 107.7)
- added C10: 100n, Capacitor_SMD:C_0603_1608Metric, F.Cu at (172.7, 155.3)
- added C11: 100n, Capacitor_SMD:C_0603_1608Metric, F.Cu at (160.5, 164.4)
- added C2: 100n, Capacitor_SMD:C_0603_1608Metric, F.Cu at (156.5, 149.8)
- added C3: 100n, Capacitor_SMD:C_0603_1608Metric, F.Cu at (180.8, 130.6)
- added C4: 100n, Capacitor_SMD:C_0603_1608Metric, F.Cu at (200.0, 110.4)
- added C5: 100n, Capacitor_SMD:C_0603_1608Metric, F.Cu at (160.5, 149.8)
- added C6: 100n, Capacitor_SMD:C_0603_1608Metric, F.Cu at (172.7, 160.3)
- added C7: 100n, Capacitor_SMD:C_0603_1608Metric, F.Cu at (172.7, 157.8)
- added C8: 1u, Capacitor_SMD:C_0805_2012Metric, F.Cu at (168.3, 162.7)
- added C9: 100n, Capacitor_SMD:C_0603_1608Metric, F.Cu at (156.5, 164.4)
- added J1: Conn_02x05_Odd_Even, Connector_IDC:IDC-Header_2x05_P2.54mm_Vertical, F.Cu at (174.6, 112.4)
- added J2: Conn_02x13_Odd_Even, Connector_IDC:IDC-Header_2x13_P2.54mm_Vertical, F.Cu at (128.9, 115.8)
- added J3: Conn_01x02, Connector_PinHeader_2.54mm:PinHeader_1x02_P2.54mm_Vertical, F.Cu at (168.4, 156.4)
- added J4: Screw_Terminal_01x02, TerminalBlock:TerminalBlock_bornier-2_P5.08mm, F.Cu at (157.7, 158.6)
- added Q1: BC857, Package_TO_SOT_SMD:SOT-23, B.Cu at (90.8, 59.4)
- added Q10: BC857, Package_TO_SOT_SMD:SOT-23, B.Cu at (112.4, 75.8)
- added Q11: BC857, Package_TO_SOT_SMD:SOT-23, B.Cu at (123.1, 59.4)
- added Q12: BC857, Package_TO_SOT_SMD:SOT-23, B.Cu at (123.2, 75.8)
- added Q13: BC857, Package_TO_SOT_SMD:SOT-23, B.Cu at (112.2, 52.4)
- added Q14: BC857, Package_TO_SOT_SMD:SOT-23, B.Cu at (112.4, 68.7)
- added Q15: BC857, Package_TO_SOT_SMD:SOT-23, B.Cu at (123.0, 52.4)
- added Q16: BC857, Package_TO_SOT_SMD:SOT-23, B.Cu at (123.2, 68.7)
- added Q17: BC857, Package_TO_SOT_SMD:SOT-23, B.Cu at (133.8, 59.4)
- added Q18: BC857, Package_TO_SOT_SMD:SOT-23, B.Cu at (134.0, 75.8)
- added Q19: BC857, Package_TO_SOT_SMD:SOT-23, B.Cu at (144.7, 59.5)
- added Q2: BC857, Package_TO_SOT_SMD:SOT-23, B.Cu at (90.8, 75.9)
- added Q20: BC857, Package_TO_SOT_SMD:SOT-23, B.Cu at (144.7, 75.8)
- added Q21: BC857, Package_TO_SOT_SMD:SOT-23, B.Cu at (133.9, 52.3)
- added Q22: BC857, Package_TO_SOT_SMD:SOT-23, B.Cu at (134.0, 68.7)
- added Q23: BC857, Package_TO_SOT_SMD:SOT-23, B.Cu at (144.7, 52.3)
- added Q24: BC857, Package_TO_SOT_SMD:SOT-23, B.Cu at (144.7, 68.7)
- added Q25: BC857, Package_TO_SOT_SMD:SOT-23, B.Cu at (155.5, 59.4)
- added Q26: BC857, Package_TO_SOT_SMD:SOT-23, B.Cu at (155.6, 75.8)
- added Q27: BC857, Package_TO_SOT_SMD:SOT-23, B.Cu at (166.3, 59.4)
- added Q28: BC857, Package_TO_SOT_SMD:SOT-23, B.Cu at (166.4, 75.8)
- added Q29: BC857, Package_TO_SOT_SMD:SOT-23, B.Cu at (155.5, 52.4)
- added Q3: BC857, Package_TO_SOT_SMD:SOT-23, B.Cu at (101.5, 59.5)
- added Q30: BC857, Package_TO_SOT_SMD:SOT-23, B.Cu at (155.6, 68.7)
- added Q31: BC857, Package_TO_SOT_SMD:SOT-23, B.Cu at (166.3, 52.3)
- added Q32: BC857, Package_TO_SOT_SMD:SOT-23, B.Cu at (166.4, 68.7)
- added Q4: BC857, Package_TO_SOT_SMD:SOT-23, B.Cu at (101.5, 75.9)
- added Q5: BC857, Package_TO_SOT_SMD:SOT-23, B.Cu at (90.7, 52.4)
- added Q6: BC857, Package_TO_SOT_SMD:SOT-23, B.Cu at (90.7, 68.7)
- added Q7: BC857, Package_TO_SOT_SMD:SOT-23, B.Cu at (101.5, 52.3)
- added Q8: BC857, Package_TO_SOT_SMD:SOT-23, B.Cu at (101.5, 68.9)
- added Q9: BC857, Package_TO_SOT_SMD:SOT-23, B.Cu at (112.2, 59.5)
- added R1: 1k, Resistor_SMD:R_0603_1608Metric, B.Cu at (19.1, 148.7)
- added R10: 1k, Resistor_SMD:R_0603_1608Metric, B.Cu at (113.3, 80.6)
- added R11: 1k, Resistor_SMD:R_0603_1608Metric, B.Cu at (50.0, 148.5)
- added R12: 1k, Resistor_SMD:R_0603_1608Metric, B.Cu at (-88.8, 106.7)
- added R13: 1k, Resistor_SMD:R_0603_1608Metric, B.Cu at (47.7, 117.3)
- added R14: 1k, Resistor_SMD:R_0603_1608Metric, B.Cu at (13.7, 119.7)
- added R15: 1k, Resistor_SMD:R_0603_1608Metric, B.Cu at (57.7, 117.0)
- added R16: 1k, Resistor_SMD:R_0603_1608Metric, B.Cu at (47.6, 150.1)
- added R17: 1k, Resistor_SMD:R_0603_1608Metric, B.Cu at (60.5, 148.8)
- added R18: 1k, Resistor_SMD:R_0603_1608Metric, B.Cu at (-78.2, 107.0)
- added R19: 1k, Resistor_SMD:R_0603_1608Metric, B.Cu at (71.8, 148.5)
- added R2: 1k, Resistor_SMD:R_0603_1608Metric, B.Cu at (-121.8, 107.5)
- added R20: 1k, Resistor_SMD:R_0603_1608Metric, B.Cu at (-67.3, 106.9)
- added R21: 1k, Resistor_SMD:R_0603_1608Metric, B.Cu at (68.5, 116.8)
- added R22: 1k, Resistor_SMD:R_0603_1608Metric, B.Cu at (57.4, 149.6)
- added R23: 1k, Resistor_SMD:R_0603_1608Metric, B.Cu at (79.4, 116.5)
- added R24: 1k, Resistor_SMD:R_0603_1608Metric, B.Cu at (68.5, 149.9)
- added R25: 1k, Resistor_SMD:R_0603_1608Metric, B.Cu at (81.7, 148.6)
- added R26: 1k, Resistor_SMD:R_0603_1608Metric, B.Cu at (-55.2, 106.9)
- added R27: 1k, Resistor_SMD:R_0603_1608Metric, B.Cu at (93.2, 148.8)
- added R28: 1k, Resistor_SMD:R_0603_1608Metric, B.Cu at (-45.5, 106.5)
- added R29: 1k, Resistor_SMD:R_0603_1608Metric, B.Cu at (89.2, 117.4)
- added R3: 1k, Resistor_SMD:R_0603_1608Metric, B.Cu at (27.8, 148.8)
- added R30: 1k, Resistor_SMD:R_0603_1608Metric, B.Cu at (111.8, 97.7)
- added R31: 1k, Resistor_SMD:R_0603_1608Metric, B.Cu at (100.8, 117.0)
- added R32: 1k, Resistor_SMD:R_0603_1608Metric, B.Cu at (90.2, 149.9)
- added R33: 1k, Resistor_SMD:R_0603_1608Metric, F.Cu at (187.4, 75.4)
- added R34: 1k, Resistor_SMD:R_0603_1608Metric, F.Cu at (185.9, 60.0)
- added R35: 1k, Resistor_SMD:R_0603_1608Metric, F.Cu at (191.0, 71.7)
- added R36: 1k, Resistor_SMD:R_0603_1608Metric, F.Cu at (187.2, 68.7)
- added R37: 1k, Resistor_SMD:R_0603_1608Metric, F.Cu at (187.1, 53.3)
- added R38: 1k, Resistor_SMD:R_0603_1608Metric, F.Cu at (186.4, 63.6)
- added R39: 1k, Resistor_SMD:R_0603_1608Metric, F.Cu at (187.5, 49.9)
- added R4: 1k, Resistor_SMD:R_0603_1608Metric, B.Cu at (-110.2, 106.7)
- added R40: 1k, Resistor_SMD:R_0603_1608Metric, F.Cu at (187.3, 56.5)
- added R5: 1k, Resistor_SMD:R_0603_1608Metric, B.Cu at (25.0, 117.2)
- added R6: 1k, Resistor_SMD:R_0603_1608Metric, B.Cu at (14.8, 149.8)
- added R7: 1k, Resistor_SMD:R_0603_1608Metric, B.Cu at (35.3, 117.5)
- added R8: 1k, Resistor_SMD:R_0603_1608Metric, B.Cu at (24.7, 149.8)
- added R9: 1k, Resistor_SMD:R_0603_1608Metric, B.Cu at (38.5, 149.0)
- added U1: 74HC595, Package_SO:SOIC-16_3.9x9.9mm_P1.27mm, F.Cu at (156.0, 35.2)
- added U10: 74HC595, Package_SO:SOIC-16_3.9x9.9mm_P1.27mm, F.Cu at (193.8, 112.0)
- added U11: 74HC595, Package_SO:SOIC-16_3.9x9.9mm_P1.27mm, F.Cu at (185.3, 112.0)
- added U2: 74HC595, Package_SO:SOIC-16_3.9x9.9mm_P1.27mm, F.Cu at (113.3, 39.2)
- added U3: 74HC595, Package_SO:SOIC-16_3.9x9.9mm_P1.27mm, F.Cu at (145.5, 92.4)
- added U4: 74HC595, Package_SO:SOIC-16_3.9x9.9mm_P1.27mm, F.Cu at (99.2, 88.2)
- added U5: ULN2803A, Package_SO:SOIC-18W_7.5x11.6mm_P1.27mm, F.Cu at (199.1, 61.8)
- added U6: 74HC595, Package_SO:SOIC-16_3.9x9.9mm_P1.27mm, F.Cu at (220.0, 62.3)
- added U7: 74HC595, Package_SO:SOIC-16_3.9x9.9mm_P1.27mm, F.Cu at (174.6, 134.2)
- added U8: 74LS165, Package_SO:SOIC-16_3.9x9.9mm_P1.27mm, F.Cu at (185.3, 123.5)
- added U9: 74AHC1G125, Package_TO_SOT_SMD:SOT-23-5, F.Cu at (192.0, 120.1)
- moved DISP13 88.9 mm to (101.6, 72.3), turned to 90 degrees
- moved DISP9 88.7 mm to (101.5, 55.9), turned to 90 degrees
- moved DISP14 80.6 mm to (123.2, 72.3), turned to 90 degrees
- moved DISP15 74.1 mm to (144.8, 72.3), turned to 90 degrees
- moved DISP5 72.5 mm to (90.8, 72.3), turned to 90 degrees
- moved DISP6 66.3 mm to (112.4, 72.3), turned to 90 degrees
- moved DISP1 59.0 mm to (90.7, 55.9), turned to 90 degrees
- moved DISP10 58.6 mm to (123.1, 55.9), turned to 90 degrees
- moved DISP11 47.0 mm to (144.7, 55.9), turned to 90 degrees
- moved DISP2 39.3 mm to (112.3, 55.9), turned to 90 degrees
- moved DISP16 38.0 mm to (166.4, 72.3), turned to 90 degrees
- moved DISP12 37.4 mm to (166.3, 55.9), turned to 90 degrees
- moved DISP7 30.1 mm to (134.0, 72.3), turned to 90 degrees
- moved DISP3 29.3 mm to (133.9, 55.9), turned to 90 degrees
- moved DISP4 24.5 mm to (155.5, 55.9), turned to 90 degrees
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Connections:
- net /A renamed /Display/A
- net /B renamed /Display/B
- net /C renamed /Display/C
- net /D renamed /Display/D
- net /DP renamed /Display/DP
- net /E renamed /Display/E
- net /F renamed /Display/F
- net /G renamed /Display/G
- DISP1 pad 3: /RCA1 -> /Display/RCA1
- DISP1 pad 8: /GCA1 -> /Display/GCA1
- DISP10 pad 3: /RCA13 -> /Display/RCA10
- DISP10 pad 8: /GCA13 -> /Display/GCA10
- DISP11 pad 3: /RCA6 -> /Display/RCA11
- DISP11 pad 8: /GCA6 -> /Display/GCA11
- DISP12 pad 3: /RCA14 -> /Display/RCA12
- DISP12 pad 8: /GCA14 -> /Display/GCA12
- DISP13 pad 3: /RCA7 -> /Display/RCA13
- DISP13 pad 8: /GCA7 -> /Display/GCA13
- DISP14 pad 3: /RCA15 -> /Display/RCA14
- DISP14 pad 8: /GCA15 -> /Display/GCA14
- DISP15 pad 3: /RCA8 -> /Display/RCA15
- DISP15 pad 8: /GCA8 -> /Display/GCA15
- DISP16 pad 3: /RCA16 -> /Display/RCA16
- DISP16 pad 8: /GCA16 -> /Display/GCA16
- DISP2 pad 3: /RCA9 -> /Display/RCA2
- DISP2 pad 8: /GCA9 -> /Display/GCA2
- DISP3 pad 3: /RCA2 -> /Display/RCA3
- DISP3 pad 8: /GCA2 -> /Display/GCA3
- DISP4 pad 3: /RCA10 -> /Display/RCA4
- DISP4 pad 8: /GCA10 -> /Display/GCA4
- DISP5 pad 3: /RCA3 -> /Display/RCA5
- DISP5 pad 8: /GCA3 -> /Display/GCA5
- DISP6 pad 3: /RCA11 -> /Display/RCA6
- DISP6 pad 8: /GCA11 -> /Display/GCA6
- DISP7 pad 3: /RCA4 -> /Display/RCA7
- DISP7 pad 8: /GCA4 -> /Display/GCA7
- DISP8 pad 3: /RCA12 -> /Display/RCA8
- DISP8 pad 8: /GCA12 -> /Display/GCA8
- DISP9 pad 3: /RCA5 -> /Display/RCA9
- DISP9 pad 8: /GCA5 -> /Display/GCA9
Routing:
- net +5V: track 0.00 -> 280.4 mm, vias 0 -> 24
- net /Display/C: track 0.00 -> 184.8 mm
- net /Display/DP: track 0.00 -> 172.7 mm
- net /Display/D: track 0.00 -> 166.0 mm
- net /Display/E: track 0.00 -> 165.8 mm
- net /Display/RCA15: track 0.00 -> 4.99 mm
- net /Display/RCA5: track 0.00 -> 4.99 mm
- net /Display/GCA9: track 0.00 -> 4.95 mm
- net /Display/RCA2: track 0.00 -> 4.95 mm
- net /Display/RCA10: track 0.00 -> 4.95 mm
- net /Display/RCA13: track 0.00 -> 4.90 mm
- net /Display/GCA1: track 0.00 -> 4.90 mm
- net /Display/RCA3: track 0.00 -> 4.89 mm
- net /Display/RCA12: track 0.00 -> 4.89 mm
- net /Display/GCA11: track 0.00 -> 4.89 mm
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Other:
- board outline added: 95 x 38.5 mm

Commit message: Update schematics
Parts:
- added ?: , , F.Cu at (113.3, 146.3)
- added REF**: MountingHole_3.2mm_M3, MountingHole:MountingHole_3.2mm_M3, F.Cu at (175.4, 49.5)
- added REF**: MountingHole_3.2mm_M3, MountingHole:MountingHole_3.2mm_M3, F.Cu at (175.4, 125.7)
- added REF**: MountingHole_3.2mm_M3, MountingHole:MountingHole_3.2mm_M3, F.Cu at (87.6, 125.7)
- C1: moved to B.Cu
- C11: value 100n -> 1u; footprint Capacitor_SMD:C_0603_1608Metric -> Capacitor_SMD:C_0805_2012Metric
- C8: value 1u -> 100n; footprint Capacitor_SMD:C_0805_2012Metric -> Capacitor_SMD:C_0603_1608Metric
- moved R2 250.1 mm to (127.3, 85.7), turned to 270 degrees
- moved R4 245.3 mm to (134.2, 85.7), turned to 270 degrees
- moved R12 234.5 mm to (144.8, 85.7), turned to 270 degrees
- moved R18 229.7 mm to (150.5, 85.7), turned to 270 degrees
- moved R20 221.9 mm to (153.6, 85.7), turned to 270 degrees
- moved R26 212.9 mm to (156.7, 85.7), turned to 270 degrees
- moved R28 206.3 mm to (159.8, 85.7), turned to 270 degrees
- moved R6 130.8 mm to (128.8, 85.7), turned to 270 degrees
- moved R14 130.5 mm to (139.7, 85.7), turned to 270 degrees
- moved R8 128.2 mm to (135.7, 85.7), turned to 270 degrees
- moved R16 117.9 mm to (146.3, 85.7), turned to 270 degrees
- moved R22 114.2 mm to (152.1, 85.7), turned to 270 degrees
- moved R24 107.8 mm to (155.2, 85.7), turned to 270 degrees
- moved C8 98.1 mm to (91.7, 101.4)
- moved R32 95.8 mm to (161.3, 85.7), turned to 270 degrees
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Connections:
- C1 pad 1: VDD -> VCC
- C10 pad 1: VDD -> VCC
- C11 pad 1: VDD -> +5V
- C2 pad 1: VDD -> VCC
- C3 pad 1: VDD -> VCC
- C4 pad 1: VDD -> VCC
- C5 pad 1: VDD -> VCC
- C6 pad 1: VDD -> VCC
- C7 pad 1: VDD -> VCC
- C8 pad 1: +5V -> VCC
- C9 pad 1: VDD -> VCC
- J1 pad 1: /CLK -> GND
- J1 pad 10: /~IN_LATCH -> /~LED_CS
- J1 pad 2: GND -> /CLK
- J1 pad 3: /DI -> GND
- J1 pad 4: GND -> /DI
- J1 pad 5: /DO -> GND
- J1 pad 6: GND -> /DO
- J1 pad 7: /~KBD_CS -> VCC
- J1 pad 8: VDD -> /~KBD_CS
- J1 pad 9: /~LED_CS -> /~IN_LATCH
- J3 pad 1: VDD -> VCC
- R33 pad 2: /Display/A -> /Display/D
- R34 pad 2: /Display/B -> /Display/DP
- R36 pad 2: /Display/D -> /Display/E
- R37 pad 2: /Display/E -> /Display/B
- R39 pad 2: /Display/G -> /Display/A
- R40 pad 2: /Display/DP -> /Display/G
- U1 pad 1: /Display/R9 -> /Display/R5
- U1 pad 10: VDD -> VCC
- U1 pad 15: /Display/G9 -> /Display/G5
- U1 pad 16: VDD -> VCC
- U1 pad 2: /Display/G10 -> /Display/G13
- U1 pad 3: /Display/R10 -> /Display/R13
- U1 pad 4: /Display/G11 -> /Display/G6
- U1 pad 5: /Display/R11 -> /Display/R6
- U1 pad 6: /Display/G12 -> /Display/G14
- U1 pad 7: /Display/R12 -> /Display/R14
- U10 pad 10: VDD -> VCC
- U10 pad 11: /~KBD_CS -> /CLK
- U10 pad 12: Net-(U10-Pad12) -> /~KBD_CS
- U10 pad 16: VDD -> VCC
- U11 pad 1: /LED2 -> /LED1
- U11 pad 10: VDD -> VCC
- U11 pad 11: /~KBD_CS -> /CLK
- U11 pad 12: Net-(U11-Pad12) -> /~KBD_CS
- U11 pad 15: /LED1 -> Net-(U11-Pad15)
- U11 pad 16: VDD -> VCC
- U11 pad 2: /LED3 -> /LED2
- U11 pad 3: Net-(U11-Pad3) -> /LED3
- U2 pad 10: VDD -> VCC
- U2 pad 14: /DI -> Net-(U2-Pad14)
- U2 pad 16: VDD -> VCC
- U2 pad 2: /Display/G2 -> /Display/G9
- U2 pad 3: /Display/R2 -> /Display/R9
- U2 pad 4: /Display/G3 -> /Display/G2
- U2 pad 5: /Display/R3 -> /Display/R2
- U2 pad 6: /Display/G4 -> /Display/G10
- U2 pad 7: /Display/R4 -> /Display/R10
- U3 pad 1: /Display/R13 -> /Display/R7
- U3 pad 10: VDD -> VCC
- U3 pad 14: Net-(U1-Pad9) -> Net-(U3-Pad14)
- U3 pad 15: /Display/G13 -> /Display/G7
- U3 pad 16: VDD -> VCC
- U3 pad 2: /Display/G14 -> /Display/G15
- U3 pad 3: /Display/R14 -> /Display/R15
- U3 pad 4: /Display/G15 -> /Display/G8
- U3 pad 5: /Display/R15 -> /Display/R8
- U3 pad 9: Net-(U3-Pad9) -> Net-(U1-Pad14)
- U4 pad 1: /Display/R5 -> /Display/R3
- U4 pad 10: VDD -> VCC
- U4 pad 14: Net-(U2-Pad9) -> Net-(U1-Pad9)
- U4 pad 15: /Display/G5 -> /Display/G3
- U4 pad 16: VDD -> VCC
- U4 pad 2: /Display/G6 -> /Display/G11
- U4 pad 3: /Display/R6 -> /Display/R11
- U4 pad 4: /Display/G7 -> /Display/G4
- U4 pad 5: /Display/R7 -> /Display/R4
- U4 pad 6: /Display/G8 -> /Display/G12
- U4 pad 7: /Display/R8 -> /Display/R12
- U4 pad 9: Net-(U1-Pad14) -> Net-(U2-Pad14)
- U5 pad 1: Net-(U5-Pad1) -> /Display/DP_DRV
- U5 pad 2: Net-(U5-Pad2) -> /Display/C_DRV
- U5 pad 3: Net-(U5-Pad3) -> /Display/E_DRV
- U5 pad 4: Net-(U5-Pad4) -> /Display/B_DRV
- U5 pad 5: Net-(U5-Pad5) -> /Display/F_DRV
- U5 pad 6: Net-(U5-Pad6) -> /Display/A_DRV
- U5 pad 7: Net-(U5-Pad7) -> /Display/G_DRV
- U5 pad 8: Net-(U5-Pad8) -> /Display/D_DRV
- U6 pad 1: Net-(U5-Pad2) -> /Display/G_DRV
- U6 pad 10: VDD -> VCC
- U6 pad 14: Net-(U3-Pad9) -> /DI
- U6 pad 15: Net-(U5-Pad1) -> /Display/D_DRV
- U6 pad 16: VDD -> VCC
- U6 pad 2: Net-(U5-Pad3) -> /Display/A_DRV
- U6 pad 3: Net-(U5-Pad4) -> /Display/F_DRV
- U6 pad 4: Net-(U5-Pad5) -> /Display/B_DRV
- U6 pad 5: Net-(U5-Pad6) -> /Display/E_DRV
- U6 pad 6: Net-(U5-Pad7) -> /Display/C_DRV
- U6 pad 7: Net-(U5-Pad8) -> /Display/DP_DRV
- U6 pad 9: Net-(U6-Pad9) -> Net-(U3-Pad14)
- U7 pad 10: VDD -> VCC
- U7 pad 11: /~KBD_CS -> /CLK
- U7 pad 12: Net-(U7-Pad12) -> /~KBD_CS
- U7 pad 16: VDD -> VCC
- U8 pad 11: /R1 -> /R2
- U8 pad 12: /R2 -> /R4
- U8 pad 13: /R3 -> /R6
- U8 pad 14: /R4 -> Net-(U8-Pad14)
- U8 pad 16: VDD -> VCC
- U8 pad 3: /R5 -> Net-(U8-Pad3)
- U8 pad 4: /R6 -> /R5
- U8 pad 5: Net-(U8-Pad5) -> /R3
- U8 pad 6: Net-(U8-Pad6) -> /R1
Routing:
- net VCC: track 0.00 -> 381.2 mm, vias 0 -> 15
- net GND: track 0.00 -> 366.9 mm, vias 0 -> 34
- net /CLK: track 0.00 -> 220.3 mm
- net /Display/A: track 0.00 -> 219.4 mm, vias 0 -> 3
- net /Display/B: track 0.00 -> 219.3 mm, vias 0 -> 3
- net /Display/G: track 0.00 -> 203.4 mm, vias 0 -> 2
- net /Display/F: track 0.00 -> 202.8 mm, vias 0 -> 3
- net +5V: track 280.4 -> 450.5 mm, vias 24 -> 32
- net /~LED_CS: track 0.00 -> 146.8 mm, vias 0 -> 10
- net /DI: track 0.00 -> 92.0 mm, vias 0 -> 2
- net /~KBD_CS: track 0.00 -> 75.3 mm, vias 0 -> 4
- net /Display/DP: track 172.7 -> 228.3 mm, vias 0 -> 3
- net Net-(Q22-Pad1): track 0.00 -> 51.9 mm
- net Net-(Q21-Pad1): track 0.00 -> 45.2 mm
- net Net-(U8-Pad9): track 0.00 -> 44.0 mm, vias 0 -> 6
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Other:
- board size 95 x 38.5 mm -> 95 x 83.2 mm

Commit message: Add production files, fix licensing
Parts:
- added G***: LOGO, keyboard:softwareless_logo58x8, F.Cu at (128.6, 84.0)
- added REF**: OSHW-Symbol_6.7x6mm_SilkScreen, Symbol:OSHW-Symbol_6.7x6mm_SilkScreen, F.Cu at (88.6, 110.0)
- added REF**: KiCad-Logo2_5mm_SilkScreen, Symbol:KiCad-Logo2_5mm_SilkScreen, F.Cu at (171.7, 114.2)
Routing:
- added copper zone on B.Cu, net GND
Other:
- board text added: "+5V"
- board text added: "2022-03-22"
- board text added: "GND"
- board text added: "Licensed under CERN-OHL-P v2 or later"
- board text added: "github.com/Aifryz/softwareless"
- board text added: "led_display v1.0"
